File: Hardware/SparkFun Qwiic ToF Imager - VL53L5CX - Mini.brd (EAGLE design)
At the start: 25.4 x 12.7 mm, 43 parts, among them J2 Vertical Qwiic Connector, J3 PTH, J4 Vertical Qwiic Connector, U1 VL53L5CX

Commit message: Fix small changes from design review. Add panel.
Parts:
- removed J3: PTH, SparkX:1X04_NO_SILK
- added J1: (no value), SparkFun-Connectors:1X04_NO_SILK
- added LOGO2: OSHW-LOGONO_SILK, SparkFun-Aesthetics:DUMMY
- added LOGO5: SPECIAL_INSTRUCTIONS-ORDERING, SparkFun-Aesthetics:ORDERING_INSTRUCTIONS
- JP1, JP2, JP5, JP6: device SparkFun:MICRO-FIDUCIAL -> SparkFun-Aesthetics:FIDUCIAL-MICRO
- JP10, JP11: device SparkFun:STAND-OFF -> SparkFun-Hardware:STAND-OFF
Connections:
- net 3.3V: now also J1.2; no longer J3.2
- net GND: now also J1.1; no longer J3.1
- net SCL: now also J1.4; no longer J3.4
- net SDA: now also J1.3; no longer J3.3
Routing:
- net SDA: track 49.7 -> 48.8 mm
- net SCL: track 48.0 -> 47.3 mm
Other:
- board text added: "2-Layer Board 0.8mm Thickness 1oz Copper"

Commit message: Add v10 production files
Parts:
- removed U$11: (no value), output:#INT#1
- added U$2: (no value), output:#LED#0
- U$5: device output:#LED#10 -> output:#INT#0
- moved U$5 5.71 mm to (13.7, 3.81), turned to 0 degrees
- moved JP7 1.27 mm to (6.35, 5.08), turned to 0 degrees
- moved U$16 0.13 mm to (19.1, 5.71)
- turned JP9 to 180 degrees
Routing:
- net N$4: track 6.49 -> 4.80 mm
- net 3.3V: track 42.9 -> 42.0 mm
Changed lines of the file:
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@@
 <layer number="44" name="Drills" color="7" fill="1" visible="no" active="yes"/>
 <layer number="45" name="Holes" color="7" fill="1" visible="yes" active="yes"/>
-<layer number="46" name="Milling" color="3" fill="1" visible="yes" active="yes"/>
+<layer number="46" name="Milling" color="3" fill="1" visible="no" active="yes"/>
 <layer number="47" name="Measures" color="7" fill="1" visible="no" active="yes"/>
 <layer number="48" name="Document" color="7" fill="1" visible="no" active="yes"/>
@@
 <attribute name="VALUE" x="10.16" y="7.112" size="0.6096" layer="27" font="vector" ratio="20" rot="R180" align="top-center"/>
 </element>
-<element name="JP9" library="SparkFun-Jumpers" package="SMT-JUMPER_2_NC_TRACE_SILK" package3d_urn="urn:adsk.eagle:package:39281/1" value="INT" x="16.51" y="3.81" smashed="yes" rot="R90">
-<attribute name="NAME" x="15.24" y="2.8575" size="0.4064" layer="25" rot="R90"/>
-<attribute name="VALUE" x="18.161" y="2.8575" size="0.4064" layer="27" rot="R90"/>
+<element name="JP9" library="SparkFun-Jumpers" package="SMT-JUMPER_2_NC_TRACE_SILK" package3d_urn="urn:adsk.eagle:package:39281/1" value="INT" x="16.51" y="3.81" smashed="yes" rot="R180">
+<attribute name="NAME" x="17.4625" y="2.54" size="0.4064" layer="25" rot="R180"/>
+<attribute name="VALUE" x="17.4625" y="5.461" size="0.4064" layer="27" rot="R180"/>
 </element>
 <element name="R3" library="SparkFun-Resistors" package="0402-TIGHT" value="1k" x="8.636" y="10.16" smashed="yes" rot="R270">
@@
 </element>
 <element name="LOGO3" library="SparkFun-Aesthetics" package="QWIIC_5.5MM" value="QWIIC_LOGO_CONNECTOR" x="20.98" y="8.89" smashed="yes" rot="MR0"/>
-<element name="JP7" library="SparkFun-Jumpers" package="SMT-JUMPER_2_NC_TRACE_SILK" package3d_urn="urn:adsk.eagle:package:39281/1" value="PWR_LED" x="6.35" y="3.81" smashed="yes" rot="R270">
-<attribute name="NAME" x="7.493" y="3.81" size="0.6096" layer="25" font="vector" ratio="20" rot="R270" align="bottom-center"/>
-<attribute name="VALUE" x="5.207" y="3.81" size="0.6096" layer="27" font="vector" ratio="20" rot="R270" align="top-center"/>
+<element name="JP7" library="SparkFun-Jumpers" package="SMT-JUMPER_2_NC_TRACE_SILK" package3d_urn="urn:adsk.eagle:package:39281/1" value="PWR_LED" x="6.35" y="5.08" smashed="yes">
+<attribute name="NAME" x="6.35" y="6.223" size="0.6096" layer="25" font="vector" ratio="20" align="bottom-center"/>
+<attribute name="VALUE" x="6.35" y="3.937" size="0.6096" layer="27" font="vector" ratio="20" align="top-center"/>
 </element>
 <element name="R6" library="SparkFun-Resistors" package="0402-TIGHT" value="47k" x="8.636" y="7.62" smashed="yes" rot="R270">
@@
 <element name="U$3" library="output" package="#3V3#13" value="" x="8.89" y="3.937" smashed="yes" rot="MR270"/>
 <element name="U$4" library="output" package="PWR12" value="" x="6.223" y="8.89" smashed="yes" rot="R90"/>
-<element name="U$5" library="output" package="#LED#10" value="" x="8.001" y="3.81" smashed="yes" rot="R90"/>
 <element name="JP10" library="SparkFun-Hardware" package="STAND-OFF" value="STAND-OFF" x="2.54" y="2.54" smashed="yes"/>
 <element name="JP11" library="SparkFun-Hardware" package="STAND-OFF" value="STAND-OFF" x="22.86" y="2.54" smashed="yes"/>
 <element name="U$8" library="output" package="#INT_#0" value="" x="16.51" y="3.556" smashed="yes" rot="MR270"/>
 <element name="U$9" library="output" package="#RST_#1" value="" x="19.05" y="3.81" smashed="yes" rot="MR270"/>
-<element name="U$16" library="output" package="#I�C#0" value="" x="19.05" y="5.588" smashed="yes" rot="R90"/>
-<element name="U$11" library="output" package="#INT#1" value="" x="14.986" y="3.81" smashed="yes" rot="R90"/>
+<element name="U$16" library="output" package="#I�C#0" value="" x="19.05" y="5.715" smashed="yes" rot="R90"/>
 <element name="U$19" library="output" package="VL53L5CX0" value="" x="17.272" y="11.684" smashed="yes" rot="MR0"/>
 <element name="U$20" library="output" package="TOF1" value="" x="11.43" y="11.684" smashed="yes" rot="MR0"/>
@@
 </element>
 <element name="LOGO5" library="SparkFun-Aesthetics" package="ORDERING_INSTRUCTIONS" value="SPECIAL_INSTRUCTIONS-ORDERING" x="30.48" y="50.8" smashed="yes"/>
+<element name="U$2" library="output" package="#LED#0" value="" x="9.271" y="5.08" smashed="yes"/>
+<element name="U$5" library="output" package="#INT#0" value="" x="13.716" y="3.81" smashed="yes"/>
 </elements>
 <signals>
@@
 <wire x1="20.544" y1="9.368" x2="20.066" y2="8.89" width="0.3048" layer="1"/>
 <wire x1="20.066" y1="8.89" x2="19.05" y2="8.89" width="0.3048" layer="1"/>
-<wire x1="7.62" y1="6.35" x2="8.89" y2="5.08" width="0.3048" layer="1"/>
-<wire x1="7.62" y1="6.35" x2="6.096" y2="6.35" width="0.3048" layer="1"/>
-<wire x1="6.096" y1="6.35" x2="5.334" y2="7.112" width="0.3048" layer="1"/>
+<wire x1="5.334" y1="7.112" x2="5.715" y2="6.731" width="0.3048" layer="1"/>
 <wire x1="3.797" y1="8.412" x2="4.923" y2="8.412" width="0.3048" layer="1"/>
 <wire x1="4.923" y1="8.412" x2="5.334" y2="8.001" width="0.3048" layer="1"/>
@@
 <wire x1="15.74" y1="6.35" x2="15.748" y2="6.342" width="0.127" layer="1"/>
 <wire x1="15.748" y1="6.342" x2="15.748" y2="5.08" width="0.3048" layer="1"/>
-<wire x1="16.51" y1="4.3307" x2="16.51" y2="4.953" width="0.127" layer="1"/>
-<wire x1="16.51" y1="4.953" x2="16.383" y2="5.08" width="0.127" layer="1"/>
-<wire x1="16.383" y1="5.08" x2="15.748" y2="5.08" width="0.127" layer="1"/>
 <wire x1="19.05" y1="8.89" x2="17.653" y2="8.89" width="0.3048" layer="1"/>
 <via x="17.653" y="8.89" extent="1-16" drill="0.3048"/>
@@
 <wire x1="12.2" y1="6.35" x2="12.2" y2="6.92241875" width="0.3048" layer="1"/>
 <contactref element="J1" pad="2"/>
-<wire x1="8.89" y1="1.27" x2="8.89" y2="3.302" width="0.3048" layer="1"/>
-<wire x1="8.89" y1="3.302" x2="8.89" y2="5.08" width="0.3048" layer="1"/>
-<wire x1="6.35" y1="3.2893" x2="8.8773" y2="3.2893" width="0.3048" layer="1"/>
-<wire x1="8.8773" y1="3.2893" x2="8.89" y2="3.302" width="0.3048" layer="1"/>
+<wire x1="8.89" y1="1.27" x2="8.89" y2="5.08" width="0.3048" layer="1"/>
+<wire x1="15.9893" y1="3.81" x2="15.9893" y2="4.8387" width="0.127" layer="1"/>
+<wire x1="15.9893" y1="4.8387" x2="15.748" y2="5.08" width="0.127" layer="1"/>
+<wire x1="6.8707" y1="5.08" x2="7.747" y2="5.08" width="0.254" layer="1"/>
+<wire x1="7.747" y1="5.08" x2="8.89" y2="5.08" width="0.254" layer="1"/>
+<wire x1="7.493" y1="6.731" x2="7.747" y2="6.477" width="0.254" layer="1"/>
+<wire x1="7.747" y1="6.477" x2="7.747" y2="5.08" width="0.254" layer="1"/>
+<wire x1="5.715" y1="6.731" x2="7.493" y2="6.731" width="0.254" layer="1"/>
 </signal>
 <signal name="GND">
@@
 <contactref element="R1" pad="2"/>
 <contactref element="JP9" pad="1"/>
-<wire x1="16.51" y1="8.39" x2="16.51" y2="6.604" width="0.127" layer="1"/>
-<wire x1="17.653" y1="5.461" x2="17.653" y2="3.683" width="0.127" layer="1"/>
-<wire x1="17.653" y1="3.683" x2="17.2593" y2="3.2893" width="0.127" layer="1"/>
-<wire x1="17.2593" y1="3.2893" x2="16.51" y2="3.2893" width="0.127" layer="1"/>
-<wire x1="16.51" y1="6.604" x2="17.653" y2="5.461" width="0.127" layer="1"/>
+<wire x1="16.51" y1="6.604" x2="16.51" y2="8.39" width="0.127" layer="1"/>
+<wire x1="17.0307" y1="3.81" x2="17.0307" y2="6.0833" width="0.127" layer="1"/>
+<wire x1="17.0307" y1="6.0833" x2="16.51" y2="6.604" width="0.127" layer="1"/>
 </signal>
 <signal name="N$3">
@@
 <contactref element="R3" pad="2"/>
 <contactref element="JP7" pad="1"/>
-<wire x1="6.35" y1="4.3307" x2="6.35" y2="5.715" width="0.127" layer="1"/>
-<via x="6.35" y="5.715" extent="1-16" drill="0.3048"/>
-<wire x1="6.35" y1="8.128" x2="6.35" y2="5.715" width="0.127" layer="16"/>
+<via x="6.35" y="6.096" extent="1-16" drill="0.3048"/>
+<wire x1="6.35" y1="8.128" x2="6.35" y2="6.096" width="0.127" layer="16"/>
 <via x="5.461" y="8.89" extent="1-16" drill="0.3048"/>
 <wire x1="8.636" y1="9.66" x2="8.616675" y2="9.66" width="0.127" layer="1"/>
@@
 <wire x1="5.461" y1="8.89" x2="5.588" y2="8.89" width="0.127" layer="16"/>
 <wire x1="5.588" y1="8.89" x2="6.35" y2="8.128" width="0.127" layer="16"/>
+<wire x1="5.8293" y1="5.08" x2="5.8293" y2="5.8293" width="0.127" layer="1"/>
+<wire x1="6.096" y1="6.096" x2="6.35" y2="6.096" width="0.127" layer="1"/>
+<wire x1="6.096" y1="6.096" x2="5.8293" y2="5.8293" width="0.127" layer="1"/>
 </signal>
 <signal name="RST">
