File: Hardware/Production/SparkFun Qwiic ToF Imager - VL53L5CX - Mini-Panel.brd (EAGLE design)
At the start: 175 x 132.6 mm, 2274 parts, among them J101 Vertical Qwiic Connector, J102 Vertical Qwiic Connector, J106 Vertical Qwiic Connector, J107 Vertical Qwiic Connector, J11 Vertical Qwiic Connector, J111 Vertical Qwiic Connector, J112 Vertical Qwiic Connector, J116 Vertical Qwiic Connector, J117 Vertical Qwiic Connector, J12 Vertical Qwiic Connector, J121 Vertical Qwiic Connector, J122 Vertical Qwiic Connector, J126 Vertical Qwiic Connector, J127 Vertical Qwiic Connector, J131 Vertical Qwiic Connector, J132 Vertical Qwiic Connector, J136 Vertical Qwiic Connector, J137 Vertical Qwiic Connector, J141 Vertical Qwiic Connector, J142 Vertical Qwiic Connector, J146 Vertical Qwiic Connector, J147 Vertical Qwiic Connector, J151 Vertical Qwiic Connector, J152 Vertical Qwiic Connector, J156 Vertical Qwiic Connector, J157 Vertical Qwiic Connector, J16 Vertical Qwiic Connector, J161 Vertical Qwiic Connector, J162 Vertical Qwiic Connector, J166 Vertical Qwiic Connector, J167 Vertical Qwiic Connector, J17 Vertical Qwiic Connector, J171 Vertical Qwiic Connector, J172 Vertical Qwiic Connector, J176 Vertical Qwiic Connector, J177 Vertical Qwiic Connector, J181 Vertical Qwiic Connector, J182 Vertical Qwiic Connector, J186 Vertical Qwiic Connector, J187 Vertical Qwiic Connector, J191 Vertical Qwiic Connector, J192 Vertical Qwiic Connector, J196 Vertical Qwiic Connector, J197 Vertical Qwiic Connector, J2 Vertical Qwiic Connector, J201 Vertical Qwiic Connector, J202 Vertical Qwiic Connector, J206 Vertical Qwiic Connector, J207 Vertical Qwiic Connector, J21 Vertical Qwiic Connector, J211 Vertical Qwiic Connector, J212 Vertical Qwiic Connector, J216 Vertical Qwiic Connector, J217 Vertical Qwiic Connector, J22 Vertical Qwiic Connector, J221 Vertical Qwiic Connector, J222 Vertical Qwiic Connector, J226 Vertical Qwiic Connector, J227 Vertical Qwiic Connector, J231 Vertical Qwiic Connector, J232 Vertical Qwiic Connector, J236 Vertical Qwiic Connector, J237 Vertical Qwiic Connector, J241 Vertical Qwiic Connector, J242 Vertical Qwiic Connector, J246 Vertical Qwiic Connector, J247 Vertical Qwiic Connector, J251 Vertical Qwiic Connector, J252 Vertical Qwiic Connector, J256 Vertical Qwiic Connector, J257 Vertical Qwiic Connector, J26 Vertical Qwiic Connector, J261 Vertical Qwiic Connector, J262 Vertical Qwiic Connector, J266 Vertical Qwiic Connector, J267 Vertical Qwiic Connector, J27 Vertical Qwiic Connector, J3 Vertical Qwiic Connector, J31 Vertical Qwiic Connector, J32 Vertical Qwiic Connector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

Commit message: Add v10 production files
Parts:
- U$10: device output:#LED#10 -> output:PWR12
- U$102, U$116, U$130, U$144, U$158, U$172, U$186, U$200, U$214, U$228, U$242, U$256, U$270, U$284, U$298, U$312, U$32, U$326, U$340, U$354, U$368, U$382, U$396, U$410, U$424, U$438, U$452, U$46, U$466, U$480, U$494, U$508, U$522, U$536, U$550, U$564, U$578, U$592, U$60, U$606, U$620, U$634, U$648, U$662, U$676, U$690, U$704, U$718, U$732, U$74, U$746, U$88: device output:#LED#10 -> output:#INT_#0
- U$103, U$117, U$12, U$131, U$145, U$159, U$173, U$187, U$201, U$215, U$229, U$243, U$257, U$271, U$285, U$299, U$313, U$327, U$33, U$341, U$355, U$369, U$383, U$397, U$411, U$425, U$439, U$453, U$467, U$47, U$481, U$495, U$509, U$523, U$537, U$551, U$565, U$579, U$593, U$607, U$61, U$621, U$635, U$649, U$663, U$677, U$691, U$705, U$719, U$733, U$747, U$75, U$89: device output:#INT_#0 -> output:#RST_#1
- U$104, U$118, U$13, U$132, U$146, U$160, U$174, U$188, U$202, U$216, U$230, U$244, U$258, U$272, U$286, U$300, U$314, U$328, U$34, U$342, U$356, U$370, U$384, U$398, U$412, U$426, U$440, U$454, U$468, U$48, U$482, U$496, U$510, U$524, U$538, U$552, U$566, U$580, U$594, U$608, U$62, U$622, U$636, U$650, U$664, U$678, U$692, U$706, U$720, U$734, U$748, U$76, U$90: device output:#RST_#1 -> output:#I�C#0
- U$105, U$119, U$133, U$14, U$147, U$161, U$175, U$189, U$203, U$217, U$231, U$245, U$259, U$273, U$287, U$301, U$315, U$329, U$343, U$35, U$357, U$371, U$385, U$399, U$413, U$427, U$441, U$455, U$469, U$483, U$49, U$497, U$511, U$525, U$539, U$553, U$567, U$581, U$595, U$609, U$623, U$63, U$637, U$651, U$665, U$679, U$693, U$707, U$721, U$735, U$749, U$77, U$91: device output:#I�C#0 -> output:VL53L5CX0
- U$106, U$120, U$134, U$148, U$15, U$162, U$176, U$190, U$204, U$218, U$232, U$246, U$260, U$274, U$288, U$302, U$316, U$330, U$344, U$358, U$36, U$372, U$386, U$400, U$414, U$428, U$442, U$456, U$470, U$484, U$498, U$50, U$512, U$526, U$540, U$554, U$568, U$582, U$596, U$610, U$624, U$638, U$64, U$652, U$666, U$680, U$694, U$708, U$722, U$736, U$750, U$78, U$92: device output:#INT#1 -> output:TOF1
- U$107, U$121, U$135, U$149, U$163, U$17, U$177, U$191, U$205, U$219, U$233, U$247, U$261, U$275, U$289, U$303, U$317, U$331, U$345, U$359, U$37, U$373, U$387, U$401, U$415, U$429, U$443, U$457, U$471, U$485, U$499, U$51, U$513, U$527, U$541, U$555, U$569, U$583, U$597, U$611, U$625, U$639, U$65, U$653, U$667, U$681, U$695, U$709, U$723, U$737, U$751, U$79, U$93: device output:VL53L5CX0 -> output:IMAGER2
- U$108, U$122, U$136, U$150, U$164, U$178, U$18, U$192, U$206, U$220, U$234, U$248, U$262, U$276, U$290, U$304, U$318, U$332, U$346, U$360, U$374, U$38, U$388, U$402, U$416, U$430, U$444, U$458, U$472, U$486, U$500, U$514, U$52, U$528, U$542, U$556, U$570, U$584, U$598, U$612, U$626, U$640, U$654, U$66, U$668, U$682, U$696, U$710, U$724, U$738, U$752, U$80, U$94: device output:TOF1 -> output:#SCL#1
- U$109, U$123, U$137, U$151, U$165, U$179, U$193, U$207, U$21, U$221, U$235, U$249, U$263, U$277, U$291, U$305, U$319, U$333, U$347, U$361, U$375, U$389, U$39, U$403, U$417, U$431, U$445, U$459, U$473, U$487, U$501, U$515, U$529, U$53, U$543, U$557, U$571, U$585, U$599, U$613, U$627, U$641, U$655, U$669, U$67, U$683, U$697, U$711, U$725, U$739, U$753, U$81, U$95: device output:IMAGER2 -> output:#SDA#0
- U$11: device output:#INT#1 -> output:#INT_#0
- U$110, U$124, U$138, U$152, U$166, U$180, U$194, U$208, U$222, U$23, U$236, U$250, U$264, U$278, U$292, U$306, U$320, U$334, U$348, U$362, U$376, U$390, U$40, U$404, U$418, U$432, U$446, U$460, U$474, U$488, U$502, U$516, U$530, U$54, U$544, U$558, U$572, U$586, U$600, U$614, U$628, U$642, U$656, U$670, U$68, U$684, U$698, U$712, U$726, U$740, U$754, U$82, U$96: device output:#SCL#1 -> output:VL53L5CX_0
- U$111, U$125, U$139, U$153, U$167, U$181, U$195, U$209, U$223, U$237, U$251, U$26, U$265, U$279, U$293, U$307, U$321, U$335, U$349, U$363, U$377, U$391, U$405, U$41, U$419, U$433, U$447, U$461, U$475, U$489, U$503, U$517, U$531, U$545, U$55, U$559, U$573, U$587, U$601, U$615, U$629, U$643, U$657, U$671, U$685, U$69, U$699, U$713, U$727, U$741, U$755, U$83, U$97: device output:#SDA#0 -> output:#LED#0
- U$112, U$126, U$140, U$154, U$168, U$182, U$196, U$210, U$224, U$238, U$252, U$266, U$27, U$280, U$294, U$308, U$322, U$336, U$350, U$364, U$378, U$392, U$406, U$42, U$420, U$434, U$448, U$462, U$476, U$490, U$504, U$518, U$532, U$546, U$56, U$560, U$574, U$588, U$602, U$616, U$630, U$644, U$658, U$672, U$686, U$70, U$700, U$714, U$728, U$742, U$756, U$84, U$98: device output:VL53L5CX_0 -> output:#INT#0
- U$2: device output:#GND#62130 -> output:#LED#0
- U$5: device output:#LED#10 -> output:#INT#0
- U$6: device output:#3V3#13 -> output:#GND#62130
- U$7: device output:PWR12 -> output:#3V3#13
- moved U$11 27.4 mm to (42.4, 3.56), flipped to the bottom, turned to 270 degrees
- moved U$2 23.0 mm to (9.27, 5.08), flipped to the top, turned to 0 degrees
- moved U$163 10.4 mm to (136.4, 24.9)
- moved U$247 10.4 mm to (136.4, 38.1)
- moved U$331 10.4 mm to (136.4, 51.3)
- moved U$415 10.4 mm to (136.4, 64.5)
- moved U$499 10.4 mm to (136.4, 77.7)
- moved U$583 10.4 mm to (136.4, 90.9)
- moved U$667 10.4 mm to (136.4, 104.1)
- moved U$751 10.4 mm to (136.4, 117.3)
- moved U$79 10.4 mm to (136.4, 11.7)
- moved U$107 10.4 mm to (32.8, 24.9)
- moved U$135 10.4 mm to (84.6, 24.9)
- moved U$149 10.4 mm to (110.5, 24.9)
- moved U$17 10.4 mm to (32.8, 11.7)
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Routing:
- net N$321: track 6.49 -> 4.80 mm
- net N$285: track 6.49 -> 4.80 mm
- net N$249: track 6.49 -> 4.80 mm
- net N$177: track 6.49 -> 4.80 mm
- net N$69: track 6.49 -> 4.80 mm
- net N$33: track 6.49 -> 4.80 mm
- net N$297: track 6.49 -> 4.80 mm
- net N$261: track 6.49 -> 4.80 mm
- net N$225: track 6.49 -> 4.80 mm
- net N$141: track 6.49 -> 4.80 mm
- net N$105: track 6.49 -> 4.80 mm
- net N$315: track 6.49 -> 4.80 mm
- net N$309: track 6.49 -> 4.80 mm
- net N$303: track 6.49 -> 4.80 mm
- net N$279: track 6.49 -> 4.80 mm
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